File: mounting.sch (KiCad schematic (older format))
At the start: 4 parts

Commit message: some routing
Parts:
- MK1, MK2, MK3, MK4: symbol Mechanical:Mounting_Hole -> robot_pcb0-rescue:Mounting_Hole-Mechanical
Changed lines of the file:
@@
 EESchema Schematic File Version 4
 LIBS:robot_pcb0-cache
-EELAYER 26 0
+EELAYER 29 0
 EELAYER END
 $Descr A4 11693 8268
@@
 $EndDescr
 $Comp
-L Mechanical:Mounting_Hole MK4
+L robot_pcb0-rescue:Mounting_Hole-Mechanical MK4
 U 1 1 5B441261
 P 5550 2950
@@
 $EndComp
 $Comp
-L Mechanical:Mounting_Hole MK2
+L robot_pcb0-rescue:Mounting_Hole-Mechanical MK2
 U 1 1 5B441268
 P 3600 2900
@@
 $EndComp
 $Comp
-L Mechanical:Mounting_Hole MK3
+L robot_pcb0-rescue:Mounting_Hole-Mechanical MK3
 U 1 1 5B44126F
 P 5550 2200
@@
 $EndComp
 $Comp
-L Mechanical:Mounting_Hole MK1
+L robot_pcb0-rescue:Mounting_Hole-Mechanical MK1
 U 1 1 5B441276
 P 3600 2200

Commit message: update
Parts:
- MK1, MK2, MK3, MK4: symbol robot_pcb0-rescue:Mounting_Hole-Mechanical -> Mechanical:MountingHole
Changed lines of the file:
@@
 $EndDescr
 $Comp
-L robot_pcb0-rescue:Mounting_Hole-Mechanical MK4
+L Mechanical:MountingHole MK4
 U 1 1 5B441261
 P 5550 2950
@@
 $EndComp
 $Comp
-L robot_pcb0-rescue:Mounting_Hole-Mechanical MK2
+L Mechanical:MountingHole MK2
 U 1 1 5B441268
 P 3600 2900
@@
 $EndComp
 $Comp
-L robot_pcb0-rescue:Mounting_Hole-Mechanical MK3
+L Mechanical:MountingHole MK3
 U 1 1 5B44126F
 P 5550 2200
@@
 $EndComp
 $Comp
-L robot_pcb0-rescue:Mounting_Hole-Mechanical MK1
+L Mechanical:MountingHole MK1
 U 1 1 5B441276
 P 3600 2200
