File: hardware/nrf52.sch (KiCad schematic (older format))
At the start: 11 parts, among them J11 NRFSWDCLK, J12 NRFSWDIO, J13 GND, J14 NRFGPIO, J15 USB_B_Mini, U8 BMD-340-A-R

Commit message: restructuring making room for firmware
Parts:
- U8: symbol BMD-340:BMD-340-A-R -> robot_pcb0-rescue:BMD-340-A-R-BMD-340
Changed lines of the file:
@@
 $EndComp
 $Comp
-L BMD-340:BMD-340-A-R U8
+L robot_pcb0-rescue:BMD-340-A-R-BMD-340 U8
 U 1 1 5CF677C5
 P 5850 3200
+AR Path="/5CF677C5" Ref="U8"  Part="1"
+AR Path="/5CF66F52/5CF677C5" Ref="U8"  Part="1"
 F 0 "U8" H 5900 5067 50  0000 C CNN
 F 1 "BMD-340-A-R" H 5900 4976 50  0000 C CNN
