File: hardware/v1_0/base.sch (KiCad schematic (older format))
At the start: 32 parts, among them J1 USB_B_Mini, J10 GPIO, J2 CAN, J3 PWR, J9 UART, P1 SWD, U1 TJA1051TK-3, U2 STM32F40X_LQFP64, U3 BMI160, Y1 8M

Commit message: preparing for work on v2 of hardware
Parts:
- U3: symbol bmi160:BMI160 -> robot_pcb0-rescue:BMI160-bmi160
Changed lines of the file:
@@
 EESchema Schematic File Version 5
-LIBS:robot_pcb0-cache
-EELAYER 29 0
+EELAYER 30 0
 EELAYER END
 $Descr A4 11693 8268
@@
 Comment3 ""
 Comment4 ""
+Comment5 ""
+Comment6 ""
+Comment7 ""
+Comment8 ""
+Comment9 ""
 $EndDescr
 $Comp
@@
 V_METER
 $Comp
-L bmi160:BMI160 U3
+L robot_pcb0-rescue:BMI160-bmi160 U3
 U 1 1 5CF27D04
 P 8700 3650
+AR Path="/5CF27D04" Ref="U3"  Part="1"
+AR Path="/5AF92F5C/5CF27D04" Ref="U3"  Part="1"
 F 0 "U3" H 8700 4365 50  0000 C CNN
 F 1 "BMI160" H 8700 4274 50  0000 C CNN
